File: hardware/herring-v4-backplane/herring-v4-backplane.kicad_sch (KiCad schematic)
At the start: 29 parts, among them J1 Conn_02x20_Odd_Even, J2 Conn_02x10_Odd_Even, J3 Conn_02x20_Odd_Even, J4 Conn_02x10_Odd_Even, J5 Conn_02x20_Odd_Even, J6 Conn_02x10_Odd_Even, J7 Conn_02x20_Odd_Even, J8 Conn_02x10_Odd_Even, J9 Jack-DC, SW1 SW_Push, SW2 SW_SPDT, U1 NE555P

Commit message: herring v4 backplane routed
Parts:
- added C6: C_Polarized_US, Capacitor_THT:CP_Radial_D5.0mm_P2.50mm, symbol Device:C_Polarized_US
- added J10, J12: Conn_02x10_Odd_Even, Connector_PinSocket_2.54mm:PinSocket_2x10_P2.54mm_Vertical, symbol Connector_Generic:Conn_02x10_Odd_Even
- added J11, J9: Conn_02x20_Odd_Even, Connector_PinSocket_2.54mm:PinSocket_2x20_P2.54mm_Vertical, symbol Connector_Generic:Conn_02x20_Odd_Even
- renumbered C2 to C1, C3 to C2, C4 to C3, C5 to C4, C6 to C5, C1 to C7, C7 to C8, J9 to J13
Connections:
- net +5V: now also C6.1, J11.1 (Pin_1), J11.2 (Pin_2), J9.1 (Pin_1), J9.2 (Pin_2); no longer J2.1 (Pin_1), J2.2 (Pin_2), J4.1 (Pin_1), J4.2 (Pin_2), J6.1 (Pin_1), J6.2 (Pin_2), J8.1 (Pin_1), J8.2 (Pin_2)
- net B0: now also J11.5 (Pin_5), J9.5 (Pin_5)
- net B1: now also J11.7 (Pin_7), J9.7 (Pin_7)
- net B10: now also J11.27 (Pin_27), J9.27 (Pin_27)
- net B11: now also J11.29 (Pin_29), J9.29 (Pin_29)
- net B12: now also J11.31 (Pin_31), J9.31 (Pin_31)
- net B13: now also J11.33 (Pin_33), J9.33 (Pin_33)
- net B14: now also J11.35 (Pin_35), J9.35 (Pin_35)
- net B16: now also J11.6 (Pin_6), J9.6 (Pin_6)
- net B17: now also J11.8 (Pin_8), J9.8 (Pin_8)
- net B18: now also J11.10 (Pin_10), J9.10 (Pin_10)
- net B19: now also J11.12 (Pin_12), J9.12 (Pin_12)
- net B2: now also J11.9 (Pin_9), J9.9 (Pin_9)
- net B20: now also J11.14 (Pin_14), J9.14 (Pin_14)
- net B21: now also J11.16 (Pin_16), J9.16 (Pin_16)
- net B22: now also J11.18 (Pin_18), J9.18 (Pin_18)
- net B23: now also J11.20 (Pin_20), J9.20 (Pin_20)
- net B24: now also J11.24 (Pin_24), J9.24 (Pin_24)
- net B25: now also J11.26 (Pin_26), J9.26 (Pin_26)
- net B26: now also J11.28 (Pin_28), J9.28 (Pin_28)
- net B27: now also J11.30 (Pin_30), J9.30 (Pin_30)
- net B28: now also J11.32 (Pin_32), J9.32 (Pin_32)
- net B29: now also J11.34 (Pin_34), J9.34 (Pin_34)
- net B3: now also J11.11 (Pin_11), J9.11 (Pin_11)
- net B30: now also J11.36 (Pin_36), J9.36 (Pin_36)
- net B32: now also J10.3 (Pin_3), J12.3 (Pin_3)
- net B33: now also J10.5 (Pin_5), J12.5 (Pin_5)
- net B34: now also J10.7 (Pin_7), J12.7 (Pin_7)
- net B35: now also J10.9 (Pin_9), J12.9 (Pin_9)
- net B36: now also J10.11 (Pin_11), J12.11 (Pin_11)
- net B37: now also J10.13 (Pin_13), J12.13 (Pin_13)
- net B38: now also J10.15 (Pin_15), J12.15 (Pin_15)
- net B39: now also J10.17 (Pin_17), J12.17 (Pin_17)
- net B4: now also J11.13 (Pin_13), J9.13 (Pin_13)
- net B40: now also J10.4 (Pin_4), J12.4 (Pin_4)
- net B41: now also J10.6 (Pin_6), J12.6 (Pin_6)
- net B42: now also J10.8 (Pin_8), J12.8 (Pin_8)
- net B43: now also J10.10 (Pin_10), J12.10 (Pin_10)
- net B44: now also J10.12 (Pin_12), J12.12 (Pin_12)
- net B45: now also J10.14 (Pin_14), J12.14 (Pin_14)
- net B46: now also J10.16 (Pin_16), J12.16 (Pin_16)
- net B47: now also J10.18 (Pin_18), J12.18 (Pin_18)
- net B5: now also J11.15 (Pin_15), J9.15 (Pin_15)
- net B6: now also J11.17 (Pin_17), J9.17 (Pin_17)
- net B7: now also J11.19 (Pin_19), J9.19 (Pin_19)
- net B8: now also J11.23 (Pin_23), J9.23 (Pin_23)
- net B9: now also J11.25 (Pin_25), J9.25 (Pin_25)
- net GND: now also C6.2, J10.19 (Pin_19), J10.20 (Pin_20), J11.21 (Pin_21), J11.22 (Pin_22), J11.3 (Pin_3), J11.39 (Pin_39), J11.4 (Pin_4), J11.40 (Pin_40), J12.19 (Pin_19), J12.20 (Pin_20), J9.21 (Pin_21), J9.22 (Pin_22), J9.3 (Pin_3), J9.39 (Pin_39), J9.4 (Pin_4), J9.40 (Pin_40)
- net /RST: now also J11.37 (Pin_37), J11.38 (Pin_38), J9.37 (Pin_37), J9.38 (Pin_38)
- new net B48: J10.1 (Pin_1), J12.1 (Pin_1), J2.1 (Pin_1), J4.1 (Pin_1), J6.1 (Pin_1), J8.1 (Pin_1)
- new net B49: J10.2 (Pin_2), J12.2 (Pin_2), J2.2 (Pin_2), J4.2 (Pin_2), J6.2 (Pin_2), J8.2 (Pin_2)
Other:
- moved on the sheet: C1, C2, C3, C4, C5, H1, H2, H3, H4, J1, J2, J3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

Commit message: Herring v4 backplane gerber files
Parts:
- removed H1, H2, H3, H4: MountingHole, MountingHole:MountingHole_2.7mm_M2.5_Pad, symbol Mechanical:MountingHole
- added H1, H2, H3, H4: MountingHole_Pad, MountingHole:MountingHole_3.2mm_M3_Pad, symbol Mechanical:MountingHole_Pad
Connections:
- net B48 is gone; now on net +5V: J10.1 (Pin_1), J12.1 (Pin_1), J2.1 (Pin_1), J4.1 (Pin_1), J6.1 (Pin_1), J8.1 (Pin_1)
- net B49 is gone; now on net +5V: J10.2 (Pin_2), J12.2 (Pin_2), J2.2 (Pin_2), J4.2 (Pin_2), J6.2 (Pin_2), J8.2 (Pin_2)
- net GND: now also H1.1, H2.1, H3.1, H4.1
Other:
- moved on the sheet: C3, C5, C6, C7, C8, D1, D2, J1, J11, J2, J3, J5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
